File: board/OBD1_Scanner/OBD1_Scanner.kicad_sch (KiCad schematic)
At the start: 0 parts

Commit message: board-fab-v1
Parts:
- added C1: 10uF/1mOhm, Capacitor_SMD:C_0603_1608Metric, symbol Device:C
- added C10: 1uF/1mOhm, Capacitor_SMD:C_0603_1608Metric, symbol Device:C
- added C11, C13, C5, C7: 10uF, Capacitor_SMD:C_0603_1608Metric, symbol Device:C
- added C12, C14, C15, C16: 0.1uF, Capacitor_SMD:C_0603_1608Metric, symbol Device:C
- added C2: 10pF, Capacitor_SMD:C_0603_1608Metric, symbol Device:C
- added C3, C4: 47uF, Capacitor_SMD:CP_Elec_6.3x7.7, symbol Device:C_Polarized
- added C6: 1uF, Capacitor_SMD:C_0603_1608Metric, symbol Device:C
- added C8: 0.1uF/1mOhm, Capacitor_SMD:C_0603_1608Metric, symbol Device:C
- added C9: 220nF/16.9mOhm, Capacitor_SMD:C_0603_1608Metric, symbol Device:C
- added D1: LED_ARGB, LEDs:LED_RGB_1210_C2890623, symbol Device:LED_ARGB
- added D4, D5: SS14, Diode_SMD:D_SMA, symbol Diode:SS14
- added D6, D7, D8: LED, LED_SMD:LED_0603_1608Metric_Pad1.05x0.95mm_HandSolder, symbol Device:LED
- added D9: 1.5SMCxxA, Diode_SMD:D_SMC, symbol Diode:1.5SMCxxA
- added H1, H2, H3, H4: MountingHole, MountingHole:MountingHole_3.2mm_M3_ISO7380_Pad_TopBottom, symbol Mechanical:MountingHole
- added J1: Conn_01x04, Connector_Molex:Molex_Mini-Fit_Jr_5569-04A2_2x02_P4.20mm_Horizontal, symbol Connector_Generic:Conn_01x04
- added J2: USB_C_Receptacle, Connector_USB:USB_C_Receptacle_G-Switch_GT-USB-7010ASV, symbol Connector:USB_C_Receptacle
- added L1: 4.7uH/31.3mOhm, Inductor_SMD:L_Changjiang_FXL0630, symbol Device:L
- added R1, R17, R3: 100k, Resistor_SMD:R_0603_1608Metric, symbol #custom:R
- added R10, R5: 10k, Resistor_SMD:R_0603_1608Metric, symbol #custom:R
- added R11: 240, Resistor_SMD:R_0603_1608Metric, symbol #custom:R
- added R12, R13: 24, Resistor_SMD:R_0603_1608Metric, symbol #custom:R
- added R14: 1k8, Resistor_SMD:R_0603_1608Metric, symbol #custom:R
- added R15, R16, R6, R7: 39, Resistor_SMD:R_0603_1608Metric, symbol #custom:R
- added R18: 82, Resistor_SMD:R_0603_1608Metric, symbol #custom:R
- added R19, R2: 100, Resistor_SMD:R_0603_1608Metric, symbol #custom:R
- added R20, R21: 5k1, Resistor_SMD:R_0603_1608Metric, symbol #custom:R
- added R4: 24k9, Resistor_SMD:R_0603_1608Metric, symbol #custom:R
- added SW1, SW2: SW_Push, Button_Switch_SMD:SW_SPST_Panasonic_EVQPL_3PL_5PL_PT_A15, symbol Switch:SW_Push
- added TP1, TP4, TP5, TP6, TP8: TestPoint, TestPoint:TestPoint_Loop_D2.60mm_Drill1.4mm_Beaded, symbol Connector:TestPoint
- added TP3: TestPoint, TestPoint:TestPoint_Pad_1.5x1.5mm, symbol Connector:TestPoint
- added U1: ESP32-S3-WROOM-1, RF_Module:ESP32-S3-WROOM-1, symbol RF_Module:ESP32-S3-WROOM-1
- added U2: LMR33630BDDA, Package_SO:Texas_HSOP-8-1EP_3.9x4.9mm_P1.27mm_ThermalVias, symbol Regulator_Switching:LMR33630BDDA
- added U3, U5: SN74LVC1T45DBV, Package_TO_SOT_SMD:SOT-23-6, symbol Logic_LevelTranslator:SN74LVC1T45DBV
- added U4: AP2112K-3.3, Package_TO_SOT_SMD:SOT-23-5, symbol Regulator_Linear:AP2112K-3.3
Connections:
- new net: R6.1, TP4.1, U3.3 (A)
- new net: D1.3 (GK), R18.2
- new net: R10.1, U5.5 (DIR)
- new net: J2.B5 (CC2), R20.2
- new net: C10.1, R17.1, U2.6 (VCC)
- new net: C2.2, R3.2, R4.1, U2.5 (FB)
- new net: J2.A5 (CC1), R21.2
- new net: TP3.1, U1.27 (IO0)
- new net: R1.2, R2.2, U2.3 (EN)
- new net: R17.2, U2.4 (PG)
- new net: C8.1, U2.7 (BOOT)
- new net: C8.2, L1.1, U2.8 (SW)
- new net: R7.1, TP6.1, U5.3 (A)
- new net: D1.2 (RK), R11.2
- new net: D1.4 (BK), R19.2
- new net: D8.2 (A), R16.2
- new net: D6.2 (A), R14.2
- new net: D7.2 (A), R15.2
- new net +12V: C1.1, C4.1, C9.1, D9.1 (A1), J1.1 (Pin_1), R1.1, R14.1, U2.2 (VIN)
- new net +3.3V: C12.1, C13.1, C15.1, C7.1, D1.1 (A), R5.2, SW1.2, U1.2 (3V3), U3.6 (VCCB), U4.5 (VOUT), U5.6 (VCCB)
- new net +5V: C14.1, C16.1, D4.1 (K), D5.1 (K), R10.2, U3.1 (VCCA), U4.1 (VIN), U4.3 (EN), U5.1 (VCCA)
- new net 5V_BUCK: C2.1, C3.1, C5.1, C6.1, D4.2 (A), L1.2, R3.1
- new net 5V_USB: D5.2 (A), J2.A4 (VBUS), J2.A9 (VBUS), J2.B4 (VBUS), J2.B9 (VBUS)
- new net D+: J2.A6 (D+), J2.B6 (D+), R12.1
- new net D-: J2.A7 (D-), J2.B7 (D-), R13.1
- new net ECU_RX: J1.3 (Pin_3), R6.2
- new net ECU_TX: J1.4 (Pin_4), R7.2
- new net GND: C1.2, C10.2, C11.2, C12.2, C13.2, C14.2, C15.2, C16.2, C3.2, C4.2, C5.2, C6.2, C7.2, C9.2, D6.1 (K), D7.1 (K), D8.1 (K), D9.2 (A2), J1.2 (Pin_2), J2.A1 (GND), J2.A12 (GND), J2.B1 (GND), J2.B12 (GND), J2.S1 (SHIELD), R20.1, R21.1, R4.2, SW2.2, TP1.1, U1.1 (GND), U1.40 (GND), U1.41 (GND), U2.1 (GND), U2.9 (GND), U3.2 (GND), U3.5 (DIR), U4.2 (GND), U5.2 (GND)
- new net LED1_B: R19.1, U1.6 (IO6)
- new net LED1_G: R18.1, U1.5 (IO5)
- new net LED1_R: R11.1, U1.4 (IO4)
- new net LED_RX: R16.1, U1.21 (IO13)
- new net LED_TX: R15.1, U1.20 (IO12)
- new net MCU_PWR_CONTROL: R2.1, U1.18 (IO10)
- new net MCU_RX: TP8.1, U1.10 (IO17), U5.4 (B)
- new net MCU_TX: TP5.1, U1.11 (IO18), U3.4 (B)
- new net RST_BUTTON: C11.1, R5.1, SW2.1, U1.3 (EN)
- new net USB_D+: R12.2, U1.14 (USB_D+)
- new net USB_D-: R13.2, U1.13 (USB_D-)
- new net USER_BUTTON: SW1.1, U1.19 (IO11)
- no-connect marks 0 -> 34
Other:
- note added: "ECU SERIAL"
- note added: "FXL0630-4R7-M"
- note added: "POWER INPUT"
- note added: "WEBENCH - says use 2x 22uF w/ ESR=3mOhm. why not a 47uF? webench also suggests 100nF w/ ESR-29.6mOhm"
- note added: "webench suggests 100k looped back to vcc . why"
